Commit message: edit s0 to p4

File: urdf/robodog_left_leg_link.xacro (robot description, xacro)
@@ -18,6 +18,6 @@
         <!-- P3 -->
         <xacro:p_link name="${name}_P3_link" length="${P3_length}" width="${P3_width}" height="${P3_height}" mass="${P3_mass}" color="${P3_color}"/>
-        <!-- S0 -->
-        <xacro:s_link name="${name}_S0_link" radius="${S0_radius}" mass="${S0_mass}" color="${S0_color}"/>
+        <!-- P4 -->
+        <xacro:r_link name="${name}_P4_link" length="${P4_length}" radius="${P4_radius}" mass="${P4_mass}" color="${P4_color}"/>
         <!-- leg-P0 -->
         <joint name="${name}_P0_joint" type="fixed">
@@ -71,9 +71,9 @@
             <child link="${name}_P3_link"/>
         </joint>
-        <!-- P3-S0 -->
-        <joint name="${name}_P3_S0_joint" type="fixed">
-            <origin xyz="${P3_length/2} 0 ${P3_height/2}" rpy="0 0 0"/>
+        <!-- P3-P4 -->
+        <joint name="${name}_P3_P4_joint" type="fixed">
+            <origin xyz="${P3_length/2} 0 ${(-P4_length/2)+(P3_height/2)}" rpy="0 0 0"/>
             <parent link="${name}_P3_link"/>
-            <child link="${name}_S0_link"/>
+            <child link="${name}_P4_link"/>
         </joint>
     </xacro:macro>

File: urdf/robodog_p_link.xacro (robot description, xacro)
@@ -15,4 +15,12 @@
                     <box size="${length} ${width} ${height}" />
                 </geometry>
+                <surface>
+                    <friction>
+                        <ode>
+                            <mu>100.0</mu> <!-- Static -->
+                            <mu2>100.0</mu2> <!-- Kinematic -->
+                        </ode>
+                    </friction>
+                </surface>
             </collision>
             <xacro:inertial_box mass="${mass}" x="${length}" y="${width}" z="${height}" origin="0 0 ${height/2}" />

File: urdf/robodog_right_leg_link.xacro (robot description, xacro)
@@ -18,6 +18,6 @@
         <!-- P3 -->
         <xacro:p_link name="${name}_P3_link" length="${P3_length}" width="${P3_width}" height="${P3_height}" mass="${P3_mass}" color="${P3_color}"/>
-        <!-- S0 -->
-        <xacro:s_link name="${name}_S0_link" radius="${S0_radius}" mass="${S0_mass}" color="${S0_color}"/>
+        <!-- P4 -->
+        <xacro:r_link name="${name}_P4_link" length="${P4_length}" radius="${P4_radius}" mass="${P4_mass}" color="${P4_color}"/>
         <!-- leg-P0 -->
         <joint name="${name}_P0_joint" type="fixed">
@@ -71,9 +71,9 @@
             <child link="${name}_P3_link"/>
         </joint>
-        <!-- P3-S0 -->
-        <joint name="${name}_P3_S0_joint" type="fixed">
-            <origin xyz="${P3_length/2} 0 ${P3_height/2}" rpy="0 0 0"/>
+        <!-- P3-P4 -->
+        <joint name="${name}_P3_P4_joint" type="fixed">
+            <origin xyz="${P3_length/2} 0 ${(-P4_length/2)+(P3_height/2)}" rpy="0 0 0"/>
             <parent link="${name}_P3_link"/>
-            <child link="${name}_S0_link"/>
+            <child link="${name}_P4_link"/>
         </joint>
     </xacro:macro>

File: urdf/robodog_urdf_parameters.xacro (robot description, xacro)
@@ -7,5 +7,5 @@
     <xacro:property name="base_width" value="0.5" />
     <xacro:property name="base_height" value="0.15" />
-    <xacro:property name="base_mass" value="0.1" />
+    <xacro:property name="base_mass" value="0.2" />
     <xacro:property name="base_color" value="teal" />
     <xacro:property name="P0_length" value="0.2" />
@@ -59,7 +59,8 @@
     <xacro:property name="P3_mass" value="0.1" />
     <xacro:property name="P3_color" value="silver" />
-    <xacro:property name="S0_radius" value="0.05" />
-    <xacro:property name="S0_mass" value="0.01" />
-    <xacro:property name="S0_color" value="magenta" />
+    <xacro:property name="P4_radius" value="0.06" />
+    <xacro:property name="P4_length" value="0.12" />
+    <xacro:property name="P4_mass" value="0.1" />
+    <xacro:property name="P4_color" value="magenta" />
     <!-- GAZEBO-->
     <material name="white">
